Commit message: enable gazebo launch and urdf

File: underwater_ws/src/underwater_sim/underwater.urdf (robot description, URDF)
Before this commit: robot underwater, 11 links, 10 joints
Links:
- removed link motor1_link
- removed link motor2_link
- removed link motor3_link
- removed link wheel1_link
- removed link wheel2_link
- removed link wheel3_link
- removed link yaw_M1_link
- added link center_link, mass 0.210; visual mesh filename=package://underwater_sim/models/meshes/centralPropeller.dae scale=0.0025 0.0025 0.0025
- link base_link: geometry collision cylinder length=0.09 radius=0.6; visual mesh filename=package://underwater_sim/models/meshes/FullRobotAssemblyS18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 scale=0.0025 0.0025 0.0025
- link shaft1_link: geometry collision cylinder length=0.4 radius=0.02; visual mesh filename=package://underwater_sim/models/meshes/motorAssembly.dae scale=0.0025 0.0025 0.0025
- link shaft2_link: geometry collision cylinder length=0.4 radius=0.02; visual mesh filename=package://underwater_sim/models/meshes/motorAssembly.dae scale=0.0025 0.0025 0.0025
- link shaft3_link: geometry collision cylinder length=0.4 radius=0.02; visual mesh filename=package://underwater_sim/models/meshes/motorAssembly.dae scale=0.0025 0.0025 0.0025
Joints:
- removed joint motor1_joint1
- removed joint motor2_joint2
- removed joint motor3_joint3
- removed joint wheel_joint1
- removed joint wheel_joint2
- removed joint wheel_joint3
- joint center_motor: child yaw_M1_link -> center_link
- joint motor1: parent motor1_link -> base_link
- joint motor2: parent motor2_link -> base_link
- joint motor3: parent motor3_link -> base_link
