Commit message: organize mesh file directory

File: underwater_ws/src/underwater_sim/urdf/ship.urdf (robot description, URDF)
Before this commit: robot ship, 2 links, 1 joints
Links:
- link ship_base_link: geometry collision mesh filename=package://underwater_sim/models/meshes/ship/ship.dae; visual mesh filename=package://underwater_sim/models/meshes/ship/ship.dae scale=0.0025 0.0025 0.0025

File: underwater_ws/src/underwater_sim/urdf/underwater.urdf (robot description, URDF)
Before this commit: robot underwater, 14 links, 13 joints
Links:
- link center_link: geometry visual mesh filename=package://underwater_sim/models/meshes/robot/CentralPropell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 scale=0.0025 0.0025 0.0025
- link cylinder1_link: geometry visual mesh filename=package://underwater_sim/models/meshes/robot/Cylinder.dae scale=0.0025 0.0025 0.0025
- link cylinder2_link: geometry visual mesh filename=package://underwater_sim/models/meshes/robot/Cylinder.dae scale=0.0025 0.0025 0.0025
- link cylinder3_link: geometry visual mesh filename=package://underwater_sim/models/meshes/robot/Cylinder.dae scale=0.0025 0.0025 0.0025
- link motorcylinder1_link: geometry visual mesh filename=package://underwater_sim/models/meshes/robot/TubeMotor.dae scale=0.0025 0.0025 0.0025
- link motorcylinder2_link: geometry visual mesh filename=package://underwater_sim/models/meshes/robot/TubeMotor.dae scale=0.0025 0.0025 0.0025
- link motorcylinder3_link: geometry visual mesh filename=package://underwater_sim/models/meshes/robot/TubeMotor.dae scale=0.0025 0.0025 0.0025
- link robot_base_link: geometry collision cylinder length=0.09 radius=0.6; visual mesh filename=package://underwater_sim/models/meshes/robot/MainBody.dae scale=0.0025 0.0025 0.0025
- link shaft1_link: geometry visual mesh filename=package://underwater_sim/models/meshes/robot/Shaft.dae scale=0.0025 0.0025 0.0025
- link shaft2_link: geometry visual mesh filename=package://underwater_sim/models/meshes/robot/Shaft.dae scale=0.0025 0.0025 0.0025
- link shaft3_link: geometry visual mesh filename=package://underwater_sim/models/meshes/robot/Shaft.dae scale=0.0025 0.0025 0.0025

Commit message: scaled ship

File: underwater_ws/src/underwater_sim/urdf/ship.urdf (robot description, URDF)
Before this commit: robot ship, 2 links, 1 joints
Links:
- link ship_base_link: geometry collision mesh filename=package://underwater_sim/models/meshes/ship/hull.dae scale=0.0025 0.0025 0.0025; visual mesh filename=package://underwater_sim/models/meshes/ship/testShip.dae scale=0.0025 0.0025 0.0025
