Commit message: Creating separate tank/ship worlds without spawning. So pretty yay

File: underwater_ws/src/underwater_sim/urdf/tank.urdf (robot description, URDF)
Before this commit: robot ship, 2 links, 1 joints
Links:
- removed link dummy_link
- added link tank_water_link, mass 95.78; collision mesh filename=package://underwater_sim/models/meshes/tank/tank_water.dae scale=0.0025 0.0025 0.0025; visual mesh filename=package://underwater_sim/models/meshes/tank/tank_water.dae scale=0.0025 0.0025 0.0025
Joints:
- removed joint dummy_joint
- added joint tank_joint: type fixed, parent tank_link, child tank_water_link, origin xyz=0 0 0

Commit message: tank test launch file

File: underwater_ws/src/underwater_sim/urdf/tank.urdf (robot description, URDF)
Before this commit: robot ship, 2 links, 1 joints
Links:
- removed link tank_link
- added link tank_base_link, mass 95.78; collision mesh filename=package://underwater_sim/models/meshes/tank/tank.dae scale=0.0025 0.0025 0.0025; visual mesh filename=package://underwater_sim/models/meshes/tank/tank.dae scale=0.0025 0.0025 0.0025
Joints:
- joint tank_joint: parent tank_link -> tank_base_link

Commit message: change imu frame and added camera to rviz

File: underwater_ws/src/underwater_sim/urdf/tank.urdf (robot description, URDF)
Before this commit: robot ship, 2 links, 1 joints
Links:
- link tank_base_link: geometry collision mesh filename=package://underwater_sim/models/meshes/tank/tank.dae scale=0.001 0.001 0.001; visual mesh filename=package://underwater_sim/models/meshes/tank/tank.dae scale=0.001 0.001 0.001
- link tank_water_link: geometry collision mesh filename=package://underwater_sim/models/meshes/tank/tank_water.dae scale=0.001 0.001 0.001; visual mesh filename=package://underwater_sim/models/meshes/tank/tank_water.dae scale=0.001 0.001 0.001

File: underwater_ws/src/underwater_sim/urdf/underwater.urdf (robot description, URDF)
Before this commit: robot underwater, 16 links, 15 joints
Joints:
- joint camera_joint: parent cylinder3_link -> cylinder2_link
- joint imu_joint: parent cylinder3_link -> cylinder2_link
