Commit message: Wow my code is so fucked, can't get water depth

File: underwater_ws/src/underwater_sim/urdf/tank_depth.xacro (robot description, xacro)
@@ -1,4 +1,5 @@
 <?xml version="1.0" ?>
-<robot name="ship" xmlns:xacro="http://ros.org/wiki/xacro">
+<robot name="tank" xmlns:xacro="http://ros.org/wiki/xacro">
+    <xacro:property name="$(arg water_depth)" default="1"/>
     <material name="transparent">
         <color rgba="1 1 1 0.4"/>
@@ -27,5 +28,5 @@
             <origin rpy="0 0 0" xyz="1.4 1.2 0"/>
             <geometry>
-                <mesh filename="package://underwater_sim/models/meshes/tank/tank_water.dae" scale="0.001 0.001 0.001"/>
+                <mesh filename="package://underwater_sim/models/meshes/tank/tank_water.dae" scale="0.001 0.001 ${water_depth*0.001}"/>
             </geometry>
             <material name="transparent"/>
@@ -34,5 +35,5 @@
             <origin rpy="0 0 0" xyz="1.4 1.2 0"/>
             <geometry>
-                <mesh filename="package://underwater_sim/models/meshes/tank/tank_water.dae" scale="0.001 0.001 0.001"/>
+                <mesh filename="package://underwater_sim/models/meshes/tank/tank_water.dae" scale="0.001 0.001 ${water_depth*0.001}"/>
             </geometry>
         </collision>
