Commit message: modify underwater robot urdf

File: underwater_ws/src/underwater_sim/urdf/underwater.urdf (robot description, URDF)
Before this commit: robot underwater, 11 links, 10 joints
Links:
- link base_link: geometry collision cylinder length=0.09 radius=0.6; visual mesh filename=package://underwater_sim/models/meshes/topPlate.dae scale=0.002 0.002 0.002
Joints:
- removed joint roll_joint
- removed joint roll_joint1
- removed joint roll_joint2
- removed joint roll_joint3
- added joint motor: type continuous, parent base_link, child yaw_M1_link, origin xyz=0.000 0 0.0005 rpy=0 0 0, axis 0 0 1, limit lower=-1 upper=1 effort=0.1 velocity=0.05
- added joint motor1: type continuous, parent motor1_link, child shaft1_link, origin xyz=.3 -.1732 0 rpy=0 0 -2.094, axis 0 1 0, limit lower=-1 upper=1 effort=0.1 velocity=0.05
- added joint motor2: type continuous, parent motor2_link, child shaft2_link, origin xyz=-.3 -.1732 0 rpy=0 0 2.094, axis 0 1 0 , limit lower=-1 upper=1 effort=0.1 velocity=0.05
- added joint motor3: type continuous, parent motor3_link, child shaft3_link, origin xyz=0 .3464 0 rpy=0 0 0, axis 0 1.5708 0, limit lower=-1 upper=1 effort=0.1 velocity=0.05

Commit message: change center joint name

File: underwater_ws/src/underwater_sim/urdf/underwater.urdf (robot description, URDF)
Before this commit: robot underwater, 11 links, 10 joints
Joints:
- removed joint motor
- added joint center_motor: type continuous, parent base_link, child yaw_M1_link, origin xyz=0.000 0 0.0005 rpy=0 0 0, axis 0 0 1, limit lower=-1 upper=1 effort=0.1 velocity=0.05

Commit message: plz

File: underwater_ws/src/underwater_sim/urdf/underwater.urdf (robot description, URDF)
Before this commit: robot underwater, 8 links, 7 joints
Links:
- added link cylinder1_link, mass 0.18; collision cylinder length=0.4 radius=0.02; visual mesh filename=package://underwater_sim/models/meshes/Cylinder.dae scale=0.0025 0.0025 0.0025
- added link cylinder2_link, mass 0.18; collision cylinder length=0.4 radius=0.02; visual mesh filename=package://underwater_sim/models/meshes/Cylinder.dae scale=0.0025 0.0025 0.0025
- added link cylinder3_link, mass 0.18; collision cylinder length=0.4 radius=0.02; visual mesh filename=package://underwater_sim/models/meshes/Cylinder.dae scale=0.0025 0.0025 0.0025
- added link motorcylinder1_link, mass 0.18; collision cylinder length=0.4 radius=0.02; visual mesh filename=package://underwater_sim/models/meshes/TubeMotor.dae scale=0.0025 0.0025 0.0025
- added link motorcylinder2_link, mass 0.18; collision cylinder length=0.4 radius=0.02; visual mesh filename=package://underwater_sim/models/meshes/TubeMotor.dae scale=0.0025 0.0025 0.0025
- added link motorcylinder3_link, mass 0.18; collision cylinder length=0.4 radius=0.02; visual mesh filename=package://underwater_sim/models/meshes/TubeMotor.dae scale=0.0025 0.0025 0.0025
- link base_link: geometry collision cylinder length=0.09 radius=0.6; visual mesh filename=package://underwater_sim/models/meshes/MainBody.dae scale=0.0025 0.0025 0.0025
- link center_link: geometry visual mesh filename=package://underwater_sim/models/meshes/CentralPropeller.dae scale=0.0025 0.0025 0.0025
Joints:
- added joint cylinder1_joint: type fixed, parent base_link, child cylinder1_link, origin xyz=0 0 0 rpy=0 0 0, axis 0 1 0, limit lower=-1 upper=1 effort=0.1 velocity=0.05
- added joint cylinder2_joint: type fixed, parent base_link, child cylinder2_link, origin xyz=0 0 0 rpy=0 0 0, axis 0 1 0, limit lower=-1 upper=1 effort=0.1 velocity=0.05
- added joint cylinder3_joint: type fixed, parent base_link, child cylinder3_link, origin xyz=0 0 0 rpy=0 0 0, axis 0 1 0, limit lower=-1 upper=1 effort=0.1 velocity=0.05
- added joint motorcylinder1_joint: type fixed, parent base_link, child motorcylinder1_link, origin xyz=0 0 0 rpy=0 0 0, axis 0 1 0, limit lower=-1 upper=1 effort=0.1 velocity=0.05
- added joint motorcylinder2_joint: type fixed, parent base_link, child motorcylinder2_link, origin xyz=0 0 0 rpy=0 0 0, axis 0 1 0, limit lower=-1 upper=1 effort=0.1 velocity=0.05
- added joint motorcylinder3_joint: type fixed, parent base_link, child motorcylinder3_link, origin xyz=0 0 0 rpy=0 0 0, axis 0 1 0, limit lower=-1 upper=1 effort=0.1 velocity=0.05
- joint motor1: origin xyz=0 .3464 0 rpy=0 0 0 -> xyz=0 0.36 0.045 rpy=0 0 0
- joint motor2: origin xyz=-.3 -.1732 0 rpy=0 0 2.094 -> xyz=-0.52 -0.3 0.045 rpy=0 0 2.094
- joint motor3: origin xyz=.3 -.1732 0 rpy=0 0 -2.094 -> xyz=0.52 -0.3 0.045 rpy=0 0 -2.094

Commit message: no

File: underwater_ws/src/underwater_sim/urdf/underwater.urdf (robot description, URDF)
Before this commit: robot underwater, 14 links, 13 joints
Joints:
- joint motor2: origin xyz=-0.52 -0.3 0.045 rpy=0 0 2.094 -> xyz=-0.31184 -0.17988 0.045 rpy=0 0 2.094
- joint motor3: origin xyz=0.52 -0.3 0.045 rpy=0 0 -2.094 -> xyz=0.31184 -0.17988 0.045 rpy=0 0 -2.094

Commit message: works

File: underwater_ws/src/underwater_sim/urdf/underwater.urdf (robot description, URDF)
Before this commit: robot underwater, 14 links, 13 joints
Links:
- link center_link: mass 0.210 -> None
- link cylinder1_link: mass 0.18 -> None; geometry visual mesh filename=package://underwater_sim/models/meshes/Cylinder.dae scale=0.0025 0.0025 0.0025
- link cylinder2_link: mass 0.18 -> None; geometry visual mesh filename=package://underwater_sim/models/meshes/Cylinder.dae scale=0.0025 0.0025 0.0025
- link cylinder3_link: mass 0.18 -> None; geometry visual mesh filename=package://underwater_sim/models/meshes/Cylinder.dae scale=0.0025 0.0025 0.0025
- link motorcylinder1_link: mass 0.18 -> None; geometry visual mesh filename=package://underwater_sim/models/meshes/TubeMotor.dae scale=0.0025 0.0025 0.0025
- link motorcylinder2_link: mass 0.18 -> None; geometry visual mesh filename=package://underwater_sim/models/meshes/TubeMotor.dae scale=0.0025 0.0025 0.0025
- link motorcylinder3_link: mass 0.18 -> None; geometry visual mesh filename=package://underwater_sim/models/meshes/TubeMotor.dae scale=0.0025 0.0025 0.0025
- link shaft1_link: mass 0.18 -> None; geometry visual mesh filename=package://underwater_sim/models/meshes/Shaft.dae scale=0.0025 0.0025 0.0025
- link shaft2_link: mass 0.18 -> None; geometry visual mesh filename=package://underwater_sim/models/meshes/Shaft.dae scale=0.0025 0.0025 0.0025
- link shaft3_link: mass 0.18 -> None; geometry visual mesh filename=package://underwater_sim/models/meshes/Shaft.dae scale=0.0025 0.0025 0.0025
- link wheel1_link: geometry collision cylinder length=0.06 radius=0.2
- link wheel2_link: geometry collision cylinder length=0.06 radius=0.2
- link wheel3_link: geometry collision cylinder length=0.06 radius=0.2
Joints:
- joint center_motor: limit lower=-1 upper=1 effort=0.1 velocity=0.05 -> lower=-1 upper=1 effort=0.0 velocity=0.00
- joint cylinder1_joint: limit lower=-1 upper=1 effort=0.1 velocity=0.05 -> lower=-1 upper=1 effort=0.0 velocity=0.00
- joint cylinder2_joint: limit lower=-1 upper=1 effort=0.1 velocity=0.05 -> lower=-1 upper=1 effort=0.0 velocity=0.00
- joint cylinder3_joint: limit lower=-1 upper=1 effort=0.1 velocity=0.05 -> lower=-1 upper=1 effort=0.0 velocity=0.00
- joint motor1: limit lower=-1 upper=1 effort=0.1 velocity=0.05 -> lower=-1 upper=1 effort=0.0 velocity=0.00
- joint motor2: limit lower=-1 upper=1 effort=0.1 velocity=0.05 -> lower=-1 upper=1 effort=0.0 velocity=0.00
- joint motor3: limit lower=-1 upper=1 effort=0.1 velocity=0.05 -> lower=-1 upper=1 effort=0.0 velocity=0.00
- joint motorcylinder1_joint: limit lower=-1 upper=1 effort=0.1 velocity=0.05 -> lower=-1 upper=1 effort=0.0 velocity=0.00
- joint motorcylinder2_joint: limit lower=-1 upper=1 effort=0.1 velocity=0.05 -> lower=-1 upper=1 effort=0.0 velocity=0.00
- joint motorcylinder3_joint: limit lower=-1 upper=1 effort=0.1 velocity=0.05 -> lower=-1 upper=1 effort=0.0 velocity=0.00
- joint wheel1_joint: limit lower=-1 upper=1 effort=0.1 velocity=0.05 -> lower=-1 upper=1 effort=0.0 velocity=0.00; origin xyz=0 0 0 rpy=0 0 0 -> xyz=0 .50 0 rpy=0 0 0
- joint wheel2_joint: limit lower=-1 upper=1 effort=0.1 velocity=0.05 -> lower=-1 upper=1 effort=0.0 velocity=0.00; origin xyz=0 0 0 rpy=0 0 0 -> xyz=0 .50 0 rpy=0 0 0
- joint wheel3_joint: limit lower=-1 upper=1 effort=0.1 velocity=0.05 -> lower=-1 upper=1 effort=0.0 velocity=0.00; origin xyz=0 0 0 rpy=0 0 0 -> xyz=0 .50 0 rpy=0 0 0

Commit message: rviz add ship

File: underwater_ws/src/underwater_sim/urdf/underwater.urdf (robot description, URDF)
Before this commit: robot underwater, 14 links, 13 joints
Links:
- removed link base_link
- added link robot_base_link, mass 0.607; collision cylinder length=0.09 radius=0.6; visual mesh filename=package://underwater_sim/models/meshes/MainBody.dae scale=0.0025 0.0025 0.0025
Joints:
- joint center_motor: parent base_link -> robot_base_link
- joint cylinder1_joint: parent base_link -> robot_base_link
- joint cylinder2_joint: parent base_link -> robot_base_link
- joint cylinder3_joint: parent base_link -> robot_base_link
- joint motor1: parent base_link -> robot_base_link
- joint motor2: parent base_link -> robot_base_link
- joint motor3: parent base_link -> robot_base_link
- joint motorcylinder1_joint: parent base_link -> robot_base_link
- joint motorcylinder2_joint: parent base_link -> robot_base_link
- joint motorcylinder3_joint: parent base_link -> robot_base_link

Commit message: urdf

File: underwater_ws/src/underwater_sim/urdf/underwater.urdf (robot description, URDF)
Before this commit: robot underwater, 14 links, 13 joints
Links:
- link center_link: mass None -> 0.0; geometry visual mesh filename=package://underwater_sim/models/meshes/CentralPropeller.dae scale=0.001 0.001 0.001
- link cylinder1_link: geometry collision cylinder length=0.09 radius=0.045; visual mesh filename=package://underwater_sim/models/meshes/Cylinder.dae scale=0.001 0.001 0.001
- link cylinder2_link: geometry collision cylinder length=0.09 radius=0.045; visual mesh filename=package://underwater_sim/models/meshes/Cylinder.dae scale=0.001 0.001 0.001
- link cylinder3_link: geometry collision cylinder length=0.09 radius=0.045; visual mesh filename=package://underwater_sim/models/meshes/Cylinder.dae scale=0.001 0.001 0.001
- link motorcylinder1_link: geometry visual mesh filename=package://underwater_sim/models/meshes/TubeMotor.dae scale=0.001 0.001 0.001
- link motorcylinder2_link: geometry visual mesh filename=package://underwater_sim/models/meshes/TubeMotor.dae scale=0.001 0.001 0.001
- link motorcylinder3_link: geometry visual mesh filename=package://underwater_sim/models/meshes/TubeMotor.dae scale=0.001 0.001 0.001
- link robot_base_link: geometry collision cylinder length=0.11 radius=0.25; visual mesh filename=package://underwater_sim/models/meshes/MainBody.dae scale=0.001 0.001 0.001
- link shaft1_link: geometry visual mesh filename=package://underwater_sim/models/meshes/Shaft.dae scale=0.001 0.001 0.001
- link shaft2_link: geometry visual mesh filename=package://underwater_sim/models/meshes/Shaft.dae scale=0.001 0.001 0.001
- link shaft3_link: geometry visual mesh filename=package://underwater_sim/models/meshes/Shaft.dae scale=0.001 0.001 0.001
- link wheel1_link: geometry collision cylinder length=0.03 radius=0.08
- link wheel2_link: geometry collision cylinder length=0.03 radius=0.08
- link wheel3_link: geometry collision cylinder length=0.03 radius=0.08
Joints:
- joint center_motor: origin xyz=0.000 0 0.0005 rpy=0 0 0 -> xyz=0.000 0 0.0000 rpy=0 0 0
- joint cylinder1_joint: origin xyz=0 0 0 rpy=0 0 0 -> xyz=.1048 .0605 -.00 rpy=0 0 0
- joint cylinder2_joint: origin xyz=0 0 0 rpy=0 0 0 -> xyz=-.1048 .0605 -.00 rpy=0 0 0
- joint cylinder3_joint: origin xyz=0 0 0 rpy=0 0 0 -> xyz=0 -.121 0 rpy=0 0 0
- joint motor1: origin xyz=0 0.36 0.045 rpy=0 0 0 -> xyz=0 0.245 0 rpy=0 0 0
- joint motor2: origin xyz=-0.31184 -0.17988 0.045 rpy=0 0 2.094 -> xyz=-.21223 -0.1224 0 rpy=0 0 2.094
- joint motor3: origin xyz=0.31184 -0.17988 0.045 rpy=0 0 -2.094 -> xyz=.21223 -0.1224 0 rpy=0 0 -2.094
- joint wheel1_joint: origin xyz=0 .50 0 rpy=0 0 0 -> xyz=0 .117 0 rpy=0 0 0
- joint wheel2_joint: origin xyz=0 .50 0 rpy=0 0 0 -> xyz=0 .117 0 rpy=0 0 0
- joint wheel3_joint: origin xyz=0 .50 0 rpy=0 0 0 -> xyz=0 .117 0 rpy=0 0 0

Commit message: urdf

File: underwater_ws/src/underwater_sim/urdf/underwater.urdf (robot description, URDF)
Before this commit: robot underwater, 14 links, 13 joints
Links:
- link robot_base_link: mass 0.607 -> 5.99

Commit message: works

File: underwater_ws/src/underwater_sim/urdf/underwater.urdf (robot description, URDF)
Before this commit: robot underwater, 14 links, 13 joints
Links:
- link center_link: geometry visual mesh filename=package://underwater_sim/models/meshes/robot/CentralPropell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 scale=0.001 0.001 0.001
- link cylinder1_link: geometry collision cylinder length=0.09 radius=0.045; visual mesh filename=package://underwater_sim/models/meshes/robot/Cylinder.dae scale=0.001 0.001 0.001
- link cylinder2_link: geometry collision cylinder length=0.09 radius=0.045; visual mesh filename=package://underwater_sim/models/meshes/robot/Cylinder.dae scale=0.001 0.001 0.001
- link cylinder3_link: geometry collision cylinder length=0.09 radius=0.045; visual mesh filename=package://underwater_sim/models/meshes/robot/Cylinder.dae scale=0.001 0.001 0.001
- link motorcylinder1_link: geometry visual mesh filename=package://underwater_sim/models/meshes/robot/TubeMotor.dae scale=0.001 0.001 0.001
- link motorcylinder2_link: geometry visual mesh filename=package://underwater_sim/models/meshes/robot/TubeMotor.dae scale=0.001 0.001 0.001
- link motorcylinder3_link: geometry visual mesh filename=package://underwater_sim/models/meshes/robot/TubeMotor.dae scale=0.001 0.001 0.001
- link robot_base_link: geometry collision cylinder length=0.11 radius=0.25; visual mesh filename=package://underwater_sim/models/meshes/robot/MainBody.dae scale=0.001 0.001 0.001
- link shaft1_link: geometry visual mesh filename=package://underwater_sim/models/meshes/robot/Shaft.dae scale=0.001 0.001 0.001
- link shaft2_link: geometry visual mesh filename=package://underwater_sim/models/meshes/robot/Shaft.dae scale=0.001 0.001 0.001
- link shaft3_link: geometry visual mesh filename=package://underwater_sim/models/meshes/robot/Shaft.dae scale=0.001 0.001 0.001

Commit message: add camera

File: underwater_ws/src/underwater_sim/urdf/underwater.urdf (robot description, URDF)
Before this commit: robot underwater, 14 links, 13 joints
Links:
- added link camera_link; collision mesh filename=package://underwater_sim/models/meshes/robot/camera.dae scale=0.001 0.001 0.001; visual mesh filename=package://underwater_sim/models/meshes/robot/camera.dae scale=0.001 0.001 0.001
Joints:
- added joint camera_joint: type fixed, parent cylinder3_link, child camera_link, origin xyz=0 -0.03 0.1 rpy=0 0 -1.5708, axis 0 1 0

Commit message: imu plugin

File: underwater_ws/src/underwater_sim/urdf/underwater.urdf (robot description, URDF)
Before this commit: robot underwater, 15 links, 14 joints
Links:
- added link imu_link; collision mesh filename=package://underwater_sim/models/meshes/robot/imu.dae scale=0.0012 0.0012 0.0012; visual mesh filename=package://underwater_sim/models/meshes/robot/imu.dae scale=0.0012 0.0012 0.0012
- link camera_link: geometry collision mesh filename=package://underwater_sim/models/meshes/robot/camera.dae scale=0.0015 0.0015 0.0015; visual mesh filename=package://underwater_sim/models/meshes/robot/camera.dae scale=0.0015 0.0015 0.0015
Joints:
- added joint imu_joint: type fixed, parent cylinder3_link, child imu_link, origin xyz=0 0 0 rpy=0 0 0, axis 0 1 0

Commit message: fix encoder plugin urdf bug

File: underwater_ws/src/underwater_sim/urdf/underwater.urdf (robot description, URDF)
Before this commit: robot underwater, 16 links, 15 joints
Links:
- link wheel1_link: mass 0 -> 0.605
- link wheel2_link: mass 0 -> 0.605
- link wheel3_link: mass 0 -> 0.605

Commit message: Cerlab logo added.

File: underwater_ws/src/underwater_sim/urdf/underwater.urdf (robot description, URDF)
Before this commit: robot underwater, 16 links, 15 joints
Links:
- added link cerlab_logo_link; visual mesh filename=package://underwater_sim/models/meshes/robot/cerlabLogo.dae scale=0.00075 0.00075 0.00075
Joints:
- added joint cerlab_logo_joint: type fixed, parent robot_base_link, child cerlab_logo_link, origin xyz=0 0 0 rpy=0 0 0, axis 0 1 0, limit lower=-1 upper=1 effort=0.0 velocity=0.00

Commit message: Does Buoyancy Work? The World Will Never Know

File: underwater_ws/src/underwater_sim/urdf/underwater.urdf (robot description, URDF)
Before this commit: robot underwater, 17 links, 16 joints
Links:
- link wheel1_link: mass 0 -> 0.308
- link wheel2_link: mass 0 -> 0.308
- link wheel3_link: mass 0 -> 0.308

Commit message: bouyancy

File: underwater_ws/src/underwater_sim/urdf/underwater.urdf (robot description, URDF)
Before this commit: robot underwater, 17 links, 16 joints
Links:
- link wheel1_link: mass 0.605 -> 0.308
- link wheel2_link: mass 0.605 -> 0.308
- link wheel3_link: mass 0.605 -> 0.308

Commit message: add thrust

File: underwater_ws/src/underwater_sim/urdf/underwater.urdf (robot description, URDF)
Before this commit: robot underwater, 17 links, 16 joints
Links:
- removed link camera_link
- removed link cerlab_logo_link
- removed link imu_link
- link center_link: mass 0.0 -> 0.0001
- link robot_base_link: geometry collision cylinder length=0.11 radius=.25; visual mesh filename=package://underwater_sim/models/meshes/robot/MainBody.dae scale=0.001 0.001 0.001
- link wheel1_link: mass 0.308 -> 0.361
- link wheel2_link: mass 0.308 -> 0.361
- link wheel3_link: mass 0.308 -> 0.361
Joints:
- removed joint camera_joint
- removed joint cerlab_logo_joint
- removed joint imu_joint
- joint center_motor: limit lower=-1 upper=1 effort=0.0 velocity=0.00 -> (none); origin xyz=0.000 0 0.0000 rpy=0 0 0 -> xyz=0.000 0 0.0001 rpy=0 0 0
- joint motor1: axis 0 1.5708 0 -> 0 1 0; limit lower=-1 upper=1 effort=0.0 velocity=0.00 -> (none)
- joint motor2: limit lower=-1 upper=1 effort=0.0 velocity=0.00 -> (none)
- joint motor3: limit lower=-1 upper=1 effort=0.0 velocity=0.00 -> (none)

Commit message: bouy

File: underwater_ws/src/underwater_sim/urdf/underwater.urdf (robot description, URDF)
Before this commit: robot underwater, 14 links, 13 joints
Links:
- added link camera_link; collision mesh filename=package://underwater_sim/models/meshes/robot/camera.dae scale=0.0015 0.0015 0.0015; visual mesh filename=package://underwater_sim/models/meshes/robot/camera.dae scale=0.0015 0.0015 0.0015
- added link cerlab_logo_link; visual mesh filename=package://underwater_sim/models/meshes/robot/cerlabLogo.dae scale=0.00075 0.00075 0.00075
- added link imu_link; collision mesh filename=package://underwater_sim/models/meshes/robot/imu.dae scale=0.0012 0.0012 0.0012; visual mesh filename=package://underwater_sim/models/meshes/robot/imu.dae scale=0.0012 0.0012 0.0012
- link center_link: mass 0.0001 -> 0.0
- link robot_base_link: geometry collision cylinder length=0.11 radius=0.25; visual mesh filename=package://underwater_sim/models/meshes/robot/MainBody.dae scale=0.001 0.001 0.001
- link wheel1_link: mass 0.361 -> 0.308
- link wheel2_link: mass 0.361 -> 0.308
- link wheel3_link: mass 0.361 -> 0.308
Joints:
- added joint camera_joint: type fixed, parent cylinder2_link, child camera_link, origin xyz=0 -0.03 0.1 rpy=0 0 -1.5708, axis 0 1 0
- added joint cerlab_logo_joint: type fixed, parent robot_base_link, child cerlab_logo_link, origin xyz=0 0 0 rpy=0 0 0, axis 0 1 0, limit lower=-1 upper=1 effort=0.0 velocity=0.00
- added joint imu_joint: type fixed, parent cylinder2_link, child imu_link, origin xyz=0 0 0 rpy=0 0 0, axis 0 1 0
- joint center_motor: limit (none) -> lower=-1 upper=1 effort=0.0 velocity=0.00; origin xyz=0.000 0 0.0001 rpy=0 0 0 -> xyz=0.000 0 0.0000 rpy=0 0 0
- joint motor1: axis 0 1 0 -> 0 1.5708 0; limit (none) -> lower=-1 upper=1 effort=0.0 velocity=0.00
- joint motor2: limit (none) -> lower=-1 upper=1 effort=0.0 velocity=0.00
- joint motor3: limit (none) -> lower=-1 upper=1 effort=0.0 velocity=0.00
