Commit message: plugin working

File: underwater_ws/src/underwater_sim/urdf/tank.xacro (robot description, xacro)
@@ -50,21 +50,21 @@
     </joint>
     <gazebo reference="tank_water_link">
-            <visual name='visual'>
-        <material>
-          <lighting>1</lighting>
-          <script>
-            <uri>file://media/materials/scripts/gazebo.material</uri>
-            <name>Gazebo/Grey</name>
-          </script>
-          <ambient>0.3 0.3 0.3 0.4</ambient>
-          <diffuse>0.7 0.7 0.7 0.4</diffuse>
-          <specular>0.01 0.01 0.01 0.4</specular>
-          <emissive>0 0 0 0.4</emissive>
-          <shader type='vertex'>
-            <normal_map>__default__</normal_map>
-          </shader>
-        </material>
-        <cast_shadows>1</cast_shadows>
-        <transparency>0.7</transparency>
+        <visual name='visual'>
+            <material>
+            <lighting>1</lighting>
+            <script>
+                <uri>file://media/materials/scripts/gazebo.material</uri>
+                <name>Gazebo/Grey</name>
+            </script>
+            <ambient>0.3 0.3 0.3 0.4</ambient>
+            <diffuse>0.7 0.7 0.7 0.4</diffuse>
+            <specular>0.01 0.01 0.01 0.4</specular>
+            <emissive>0 0 0 0.4</emissive>
+            <shader type='vertex'>
+                <normal_map>__default__</normal_map>
+            </shader>
+            </material>
+            <cast_shadows>1</cast_shadows>
+            <transparency>0.7</transparency>
         </visual>
     </gazebo>

Commit message: transparent water in tank

File: underwater_ws/src/underwater_sim/urdf/tank.xacro (robot description, xacro)
@@ -50,10 +50,10 @@
     </joint>
     <gazebo reference="tank_water_link">
-        <visual name='visual'>
+        <!--<visual name='visual'>
             <material>
             <lighting>1</lighting>
             <script>
                 <uri>file://media/materials/scripts/gazebo.material</uri>
-                <name>Gazebo/Grey</name>
+                <name>Gazebo/Black</name>
             </script>
             <ambient>0.3 0.3 0.3 0.4</ambient>
@@ -66,6 +66,10 @@
             </material>
             <cast_shadows>1</cast_shadows>
-            <transparency>0.7</transparency>
-        </visual>
+            <transparency>0</transparency>
+        </visual>-->
+        <material>Gazebo/BlueTransparent</material>
+    </gazebo>
+    <gazebo reference="tank_base_link">
+        <material>Gazebo/GreyTransparent</material>
     </gazebo>
 </robot>
