Commit message: hope

File: underwater_ws/src/UGazebo/urdf/underwater.urdf (robot description, URDF)
Before this commit: robot underwater, 14 links, 13 joints
Links:
- added link flipper1_link
- added link flipper2_link
- added link flipper3_link
- added link shaft1_link_fixed
- added link shaft2_link_fixed
- added link shaft3_link_fixed
Joints:
- added joint flipper1_joint: type fixed, parent shaft1_link, child flipper1_link, origin xyz=0 .0475 0 rpy=0 0 0, axis 0 1 0, limit lower=-1 upper=1 effort=0.0 velocity=0.00
- added joint flipper2_joint: type fixed, parent shaft2_link, child flipper2_link, origin xyz=0 .0475 0 rpy=0 0 0, axis 0 1 0, limit lower=-1 upper=1 effort=0.0 velocity=0.00
- added joint flipper3_joint: type fixed, parent shaft3_link, child flipper3_link, origin xyz=0 .0475 0 rpy=0 0 0, axis 0 1 0, limit lower=-1 upper=1 effort=0.0 velocity=0.00
- added joint motor1_fixed: type fixed, parent robot_base_link, child shaft1_link_fixed, origin xyz=0 0.245 0 rpy=0 0 0, axis 0 1 0
- added joint motor2_fixed: type fixed, parent robot_base_link, child shaft2_link_fixed, origin xyz=-.21223 -0.1224 0 rpy=0 0 2.094, axis 0 1 0 
- added joint motor3_fixed: type fixed, parent robot_base_link, child shaft3_link_fixed, origin xyz=.21223 -0.1224 0 rpy=0 0 -2.094, axis 0 1 0
- joint motor1: axis 0 1.5708 0 -> 0 1 0

Commit message: wooh

File: underwater_ws/src/UGazebo/urdf/underwater.urdf (robot description, URDF)
Before this commit: robot underwater, 20 links, 19 joints
Links:
- link robot_base_link: geometry collision cylinder length=0.11 radius=.25; visual mesh filename=package://underwater_sim/models/meshes/robot/MainBody.dae scale=0.001 0.001 0.001
Joints:
- joint center_motor: type continuous -> fixed

Commit message: ugazebo

File: underwater_ws/src/UGazebo/urdf/underwater.urdf (robot description, URDF)
Before this commit: robot underwater, 20 links, 19 joints
Links:
- removed link flipper1_link
- removed link flipper2_link
- removed link flipper3_link
- removed link shaft1_link_fixed
- removed link shaft2_link_fixed
- removed link shaft3_link_fixed
- link center_link: mass 0.0 -> 0.001
Joints:
- removed joint flipper1_joint
- removed joint flipper2_joint
- removed joint flipper3_joint
- removed joint motor1_fixed
- removed joint motor2_fixed
- removed joint motor3_fixed
- joint center_motor: origin xyz=0.000 0 0.0000 rpy=0 0 0 -> xyz=0.000 0 0.0001 rpy=0 0 0; type fixed -> continuous

Commit message: added stuff

File: underwater_ws/src/UGazebo/urdf/underwater.urdf (robot description, URDF)
Before this commit: robot underwater, 14 links, 13 joints
Links:
- link center_link: mass 0.001 -> 0.0001

Commit message: combine urdfs and attach plugins using same api with arduino

File: underwater_ws/src/UGazebo/urdf/underwater.urdf (robot description, URDF)
Before this commit: robot underwater, 17 links, 16 joints
Links:
- removed link camera_link
- removed link cerlab_logo_link
- removed link imu_link
- link center_link: mass 0.0000 -> 0.0001
- link robot_base_link: geometry collision cylinder length=0.11 radius=.25; visual mesh filename=package://underwater_sim/models/meshes/robot/MainBody.dae scale=0.001 0.001 0.001
- link wheel1_link: mass 0.308 -> 0.361
- link wheel2_link: mass 0.308 -> 0.361
- link wheel3_link: mass 0.308 -> 0.361
Joints:
- removed joint camera_joint
- removed joint cerlab_logo_joint
- removed joint imu_joint
- removed joint motor_1
- removed joint motor_2
- removed joint motor_3
- added joint motor1: type continuous, parent robot_base_link, child shaft1_link, origin xyz=0 0.245 0 rpy=0 0 0, axis 0 1 0
- added joint motor2: type continuous, parent robot_base_link, child shaft2_link, origin xyz=-.21223 -0.1224 0 rpy=0 0 2.094, axis 0 1 0 
- added joint motor3: type continuous, parent robot_base_link, child shaft3_link, origin xyz=.21223 -0.1224 0 rpy=0 0 -2.094, axis 0 1 0
- joint center_motor: limit lower=-1 upper=1 effort=0.0 velocity=0.00 -> (none)
